File: Production Files/HTU21D Breakout-Panel-v12.brd (EAGLE design)
At the start: 123.4 x 123.4 mm, 640 parts, among them U1 HTU21D, U10 HTU21D, U11 HTU21D, U12 HTU21D, U13 HTU21D, U14 HTU21D, U15 HTU21D, U16 HTU21D, U17 HTU21D, U18 HTU21D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

Commit message: Recreated Panel
Parts:
- renumbered E$6 to E$5
Other:
- outline, holes or cut-outs redrawn
- board text added: "v12"
- board text removed: "v11"
